File: Hardware/Torsher/Torsher.kicad_pcb (KiCad board)
At the start: 2 copper layers, 60 x 60 mm, 20 parts, among them J1 Bx, J2 5V+, J3 SUP_DIODE, J4 RELAY, J5 SUP_RES, J6 DS 3231, J7 5V-, Q1 2SC945, U1 WeMos D1 Mini, U2 L7805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

Commit message: Add files via upload
Parts:
- removed G*** (x2): LOGO, LOGO
- added Strogg engineer logo: LOGO, LOGO, F.Cu at (145.6, 116.1)
- added Strogg logo: LOGO, LOGO, F.Cu at (101.0, 109.2)
- C1: value 0.1Mf -> 100n
- C2: value 10Mf -> 10Mф
- J2: value 5V+ -> 5B+
- J3: value SUP_DIODE -> Диод
- J4: value RELAY -> Реле
- J5: value SUP_RES -> Рез
- J7: value 5V- -> 5B-
- Q1: value 2SC945 -> C945
- moved R3 3.10 mm to (116.4, 124.4)
- moved R1 3.10 mm to (124.5, 109.1)
- moved R2 3.10 mm to (120.5, 124.3)
- moved R4 3.10 mm to (129.2, 124.3)
Routing:
- net GND: track 0.00 -> 151.1 mm
- net 5V: track 0.00 -> 147.6 mm
- net 5Vin: track 0.00 -> 77.3 mm
- net Net-(U3-ADJ): track 0.00 -> 56.1 mm
- net Net-(J5-Pin_2): track 0.00 -> 50.0 mm
- net relay_in1: track 0.00 -> 48.3 mm
- net sda: track 0.00 -> 43.3 mm
- net scl: track 0.00 -> 41.6 mm
- net relay_in2: track 0.00 -> 33.9 mm
- net sdi: track 0.00 -> 33.5 mm
- net Net-(J5-Pin_1): track 0.00 -> 29.1 mm
- net Net-(U1-A0): track 0.00 -> 25.0 mm
- net Net-(Q1-Pad1): track 0.00 -> 19.7 mm
- net D4: track 0.00 -> 15.9 mm
- added copper zone on B.Cu, net GND
- added copper zone on F.Cu, net GND
Other:
- outline, holes or cut-outs redrawn
- board text added: "github.com/coprolitebbs/Torsher"
