File: Hardware/Torsher/Torsher.kicad_pcb (KiCad board)
At the start: 2 copper layers, 60 x 60 mm, 20 parts, among them J1 Bx, J2 5B+, J3 Диод, J4 Реле, J5 Рез, J6 DS 3231, J7 5B-, Q1 C945, U1 WeMos D1 Mini, U2 L7805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

Commit message: Add files via upload
Parts:
- C2: value 10Mф -> 10Mf
- J2: value 5B+ -> 5V+
- J3: value Диод -> diode
- J4: value Реле -> RELAY
- J5: value Рез -> res
- J7: value 5B- -> 5V-
- Q1: value C945 -> 2SC945
Connections:
- J6 pad 5: 5V -> 3-3v
- U1 pad 8: unconnected-(U1-3V3-Pad8) -> 3-3v
Routing:
- net 3-3v: track 0.00 -> 27.7 mm
Changed lines of the file:
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@@
   (net 6 "unconnected-(U1-MOSI{slash}D7-Pad6)")
   (net 7 "unconnected-(U1-CS{slash}D8-Pad7)")
-  (net 8 "unconnected-(U1-3V3-Pad8)")
+  (net 8 "3-3v")
   (net 9 "5V")
   (net 10 "GND")
@@
       (net 7 "unconnected-(U1-CS{slash}D8-Pad7)") (pinfunction "CS/D8") (pintype "bidirectional+no_connect"))
     (pad "8" thru_hole oval (at 0 17.78) (size 2 1.6) (drill 1) (layers "*.Cu" "*.Mask")
-      (net 8 "unconnected-(U1-3V3-Pad8)") (pinfunction "3V3") (pintype "power_out+no_connect"))
+      (net 8 "3-3v") (pinfunction "3V3") (pintype "power_out"))
     (pad "9" thru_hole oval (at 22.86 17.78) (size 2 1.6) (drill 1) (layers "*.Cu" "*.Mask")
       (net 9 "5V") (pinfunction "5V") (pintype "power_in"))
@@
         (effects (font (size 1 1) (thickness 0.15)))
     )
-    (fp_text value "Реле" (at 0.1 -2.48) (layer "F.SilkS")
+    (fp_text value "RELAY" (at 0.1 -2.48) (layer "F.SilkS")
         (effects (font (size 1 1) (thickness 0.15)))
     )
@@
         (effects (font (size 1 1) (thickness 0.15)))
     )
-    (fp_text value "5B+" (at 0.1 -2.52 90) (layer "F.SilkS")
+    (fp_text value "5V+" (at 0.1 -2.52 90) (layer "F.SilkS")
         (effects (font (size 1 1) (thickness 0.15)))
     )
@@
         (effects (font (size 1 1) (thickness 0.1)) (justify left bottom))
     )
-    (fp_text user "5B+" (at 1.905 10.795 -90 unlocked) (layer "F.SilkS")
+    (fp_text user "3.3B+" (at 1.905 10.795 -90 unlocked) (layer "F.SilkS")
         (effects (font (size 1 1) (thickness 0.1)) (justify left bottom))
     )
@@
       (net 13 "sda") (pinfunction "Pin_4") (pintype "passive"))
     (pad "5" thru_hole oval (at 0 10.16 270) (size 1.7 1.7) (drill 1) (layers "*.Cu" "*.Mask")
-      (net 9 "5V") (pinfunction "Pin_5") (pintype "passive"))
+      (net 8 "3-3v") (pinfunction "Pin_5") (pintype "passive"))
     (model "${KICAD6_3DMODEL_DIR}/Connector_PinSocket_2.54mm.3dshapes/PinSocket_1x05_P2.54mm_Vertical.wrl"
       (offset (xyz 0 0 0))
@@
         (effects (font (size 1 1) (thickness 0.15)))
     )
-    (fp_text value "Рез" (at -0.6 -3.06 180) (layer "F.SilkS")
+    (fp_text value "res" (at -0.6 -3.06 180) (layer "F.SilkS")
         (effects (font (size 1 1) (thickness 0.15)))
     )
@@
         (effects (font (size 0.8 0.8) (thickness 0.15)))
     )
-    (fp_text value "C945" (at 0.16 -2.7 90) (layer "F.SilkS") hide
+    (fp_text value "2SC945" (at 0.16 -2.7 90) (layer "F.SilkS") hide
         (effects (font (size 0.787402 0.787402) (thickness 0.15)))
     )
@@
         (effects (font (size 1 1) (thickness 0.15)))
     )
-    (fp_text value "10Mф" (at 5.0051 -0.5 90) (layer "F.SilkS")
+    (fp_text value "10Mf" (at 5.0051 -0.5 90) (layer "F.SilkS")
         (effects (font (size 1 1) (thickness 0.15)))
     )
@@
         (effects (font (size 1 1) (thickness 0.15)))
     )
-    (fp_text value "5B-" (at 2.5 2.98 180) (layer "F.SilkS")
+    (fp_text value "5V-" (at 2.5 2.98 180) (layer "F.SilkS")
         (effects (font (size 1 1) (thickness 0.15)))
     )
@@
         (effects (font (size 1 1) (thickness 0.15)))
     )
-    (fp_text value "Диод" (at 3.7 2.14 180) (layer "F.SilkS")
+    (fp_text value "diode" (at 3.7 2.14 180) (layer "F.SilkS")
         (effects (font (size 1 1) (thickness 0.15)))
     )
@@
   (segment (start 120.5 124.32) (end 120.5 117.395) (width 0.25) (layer "B.Cu") (net 2))
   (segment (start 111.1 103.5) (end 111.1 104.6251) (width 0.25) (layer "B.Cu") (net 2))
+  (segment (start 96.14 98.04) (end 96.14 97.6) (width 0.4) (layer "F.Cu") (net 8))
+  (segment (start 111.1 118.74) (end 110.44 118.74) (width 0.4) (layer "F.Cu") (net 8))
+  (segment (start 108.7 117) (end 108.7 110.6) (width 0.4) (layer "F.Cu") (net 8))
+  (segment (start 110.44 118.74) (end 108.7 117) (width 0.4) (layer "F.Cu") (net 8))
+  (segment (start 108.7 110.6) (end 96.14 98.04) (width 0.4) (layer "F.Cu") (net 8))
   (segment (start 101.46 93.5) (end 101.5 93.46) (width 0.4) (layer "F.Cu") (net 9))
   (segment (start 100.3 84.2) (end 102.62 81.88) (width 0.4) (layer "F.Cu") (net 9))
@@
   (segment (start 99.2949 116.4949) (end 104.06 121.26) (width 0.4) (layer "F.Cu") (net 9))
   (segment (start 98.92 93.5) (end 101.46 93.5) (width 0.4) (layer "F.Cu") (net 9))
-  (segment (start 98.92 94.0875) (end 98.92 94.6751) (width 0.4) (layer "F.Cu") (net 9))
   (segment (start 105.5 121.26) (end 132.5651 121.26) (width 0.4) (layer "F.Cu") (net 9))
-  (segment (start 97.1702 96.4249) (end 98.92 94.6751) (width 0.4) (layer "F.Cu") (net 9))
   (segment (start 101.5 93.46) (end 101.5 92.4) (width 0.4) (layer "F.Cu") (net 9))
   (segment (start 135.53 86.04) (end 135.53 87.3176) (width 0.4) (layer "F.Cu") (net 9))
@@
   (segment (start 105.2387 121.26) (end 105.5 121.26) (width 0.25) (layer "F.Cu") (net 9))
   (segment (start 137.9506 89.7382) (end 141.0982 89.7382) (width 0.4) (layer "F.Cu") (net 9))
-  (segment (start 96.14 97.6) (end 96.14 96.4249) (width 0.4) (layer "F.Cu") (net 9))
-  (segment (start 96.14 96.4249) (end 97.1702 96.4249) (width 0.4) (layer "F.Cu") (net 9))
   (segment (start 98.92 93.5) (end 98.92 94.0875) (width 0.25) (layer "F.Cu") (net 9))
   (segment (start 100.3 91.2) (end 100.3 84.2) (width 0.4) (layer "F.Cu") (net 9))
@@
   (segment (start 101.5 92.4) (end 100.3 91.2) (width 0.4) (layer "F.Cu") (net 9))
   (segment (start 129.2 109.08) (end 129.2 115.1) (width 0.4) (layer "B.Cu") (net 9))
-  (segment (start 96.14 97.6) (end 96.14 98.7751) (width 0.4) (layer "B.Cu") (net 9))
+  (segment (start 97.43 98.83) (end 99.2949 100.6949) (width 0.4) (layer "B.Cu") (net 9))
   (segment (start 133.96 118.74) (end 136.2 118.74) (width 0.4) (layer "B.Cu") (net 9))
-  (segment (start 99.2949 116.1) (end 99.2949 101.93) (width 0.4) (layer "B.Cu") (net 9))
+  (segment (start 99.2949 100.6949) (end 99.2949 116.1) (width 0.4) (layer "B.Cu") (net 9))
   (segment (start 135.53 87.3176) (end 135.53 86.04) (width 0.4) (layer "B.Cu") (net 9))
   (segment (start 132.84 118.74) (end 133.96 118.74) (width 0.4) (layer "B.Cu") (net 9))
   (segment (start 129.2 115.1) (end 132.84 118.74) (width 0.4) (layer "B.Cu") (net 9))
+  (segment (start 97.7 93.5) (end 97.43 93.77) (width 0.4) (layer "B.Cu") (net 9))
+  (segment (start 98.92 93.5) (end 97.7 93.5) (width 0.4) (layer "B.Cu") (net 9))
   (segment (start 136.2 87.9876) (end 135.53 87.3176) (width 0.4) (layer "B.Cu") (net 9))
-  (segment (start 99.2949 101.93) (end 96.14 98.7751) (width 0.4) (layer "B.Cu") (net 9))
   (segment (start 136.2 118.74) (end 136.2 87.9876) (width 0.4) (layer "B.Cu") (net 9))
+  (segment (start 97.43 93.77) (end 97.43 98.83) (width 0.4) (layer "B.Cu") (net 9))
   (segment (start 108.9 84.42) (end 108.9 83.2449) (width 0.25) (layer "F.Cu") (net 10))
   (segment (start 128.8338 122.3662) (end 135.8338 122.3662) (width 0.25) (layer "F.Cu") (net 10))
