File: Hardware/Torsher/Torsher.kicad_sch (KiCad schematic)
At the start: 18 parts, among them J1 Bx, J2 5V+, J3 SUP_DIODE, J4 RELAY, J5 SUP_RES, J6 DS 3231, J7 5V-, Q1 2SC945, U1 WeMos D1 Mini, U2 L7805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

Commit message: Add files via upload
Parts:
- J3: value SUP_DIODE -> diode
- J5: value SUP_RES -> res
Changed lines of the file:
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@@
       (effects (font (size 1.27 1.27)) (justify left))
     )
-    (property "Value" "SUP_RES" (at 135.89 34.29 90)
+    (property "Value" "res" (at 135.89 34.29 90)
       (effects (font (size 1.27 1.27)) (justify left))
     )
@@
       (effects (font (size 1.27 1.27)) (justify left))
     )
-    (property "Value" "SUP_DIODE" (at 118.11 22.86 90)
-      (effects (font (size 1.27 1.27)) (justify left))
-    )
+    (property "Value" "diode" (at 118.11 22.86 90)
+      (effects (font (size 1.27 1.27)) (justify left))
+    )

Commit message: Add files via upload
Connections:
- net +5V: no longer J6.5 (Pin_5)
- net 3-3v: now reaches U1.8 (3V3)
- net 3-3v: now also J6.5 (Pin_5)
- no-connect marks 10 -> 9
Changed lines of the file:
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@@
   (no_connect (at 39.37 68.58))
   (no_connect (at 59.69 78.74))
-  (no_connect (at 52.07 48.26))
   (wire (pts (xy 128.27 63.5) (xy 128.27 62.23))
     (stroke (width 0) (type default))
@@
     (stroke (width 0) (type default))
   )
+  (wire (pts (xy 52.07 44.45) (xy 52.07 48.26))
+    (stroke (width 0) (type default))
+  )
   (wire (pts (xy 90.17 121.92) (xy 85.09 121.92))
     (stroke (width 0) (type default))
@@
     (stroke (width 0) (type default))
   )
-  (wire (pts (xy 154.94 31.75) (xy 154.94 34.29))
+  (wire (pts (xy 154.94 31.75) (xy 154.94 39.37))
     (stroke (width 0) (type default))
   )
@@
     )
   )
+  (global_label "3-3v" (shape input) (at 52.07 44.45 0) (fields_autoplaced)
+    (effects (font (size 1.27 1.27)) (justify left))
+    (property "Intersheetrefs" "${INTERSHEET_REFS}" (at 59.9348 44.45 0)
+      (effects (font (size 1.27 1.27)) (justify left) hide)
+    )
+  )
   (global_label "5Vin" (shape input) (at 66.04 111.76 180) (fields_autoplaced)
     (effects (font (size 1.27 1.27)) (justify right))
@@
     (effects (font (size 1.27 1.27)) (justify right))
     (property "Intersheetrefs" "${INTERSHEET_REFS}" (at 118.11 73.7233 90)
+      (effects (font (size 1.27 1.27)) (justify right) hide)
+    )
+  )
+  (global_label "3-3v" (shape input) (at 154.94 39.37 270) (fields_autoplaced)
+    (effects (font (size 1.27 1.27)) (justify right))
+    (property "Intersheetrefs" "${INTERSHEET_REFS}" (at 154.94 47.2348 90)
       (effects (font (size 1.27 1.27)) (justify right) hide)
     )
@@
         )
       )
-    )
-  )
-  (symbol (lib_id "power:+5V") (at 154.94 34.29 180) (unit 1)
-    (in_bom yes) (on_board yes) (dnp no) (fields_autoplaced)
-    (property "Reference" "#PWR014" (at 154.94 30.48 0)
-      (effects (font (size 1.27 1.27)) hide)
-    )
-    (property "Value" "+5V" (at 154.94 39.37 0)
-      (effects (font (size 1.27 1.27)))
-    )
-    (property "Footprint" "" (at 154.94 34.29 0)
-      (effects (font (size 1.27 1.27)) hide)
-    )
-    (property "Datasheet" "" (at 154.94 34.29 0)
-      (effects (font (size 1.27 1.27)) hide)
-    )
-    (pin "1")
-    (instances
-      (project "Torsher"
-        (path "/5758249e-256d-4032-b648-57ef0b5fd8e9"
-          (reference "#PWR014") (unit 1)
-        )
-      )
